File: WASP_filter/wasp/wasp_0.5.sch (KiCad schematic (older format))
At the start: 61 parts, among them J1 INPUT_SWT, J2 RES_POT, J3 FLT_MODE_SWT, J4 CUT_POT, J5 OUT_SWT, J6 CV, J7 Eurorack_16_pin, U1 4069, U2 LM13700, U3 AMS1117-5.0

Commit message: Yousynth ADSR layed out in Kicad, WASP reworked for more compact layout, FC more VCAs layed out
Parts:
- R2, R4: footprint Resistor_THT:R_Axial_DIN0207_L6.3mm_D2.5mm_P2.54mm_Vertical -> Resistor_THT:R_Axial_DIN0207_L6.3mm_D2.5mm_P10.16mm_Horizontal
- R25, R29: footprint Resistor_THT:R_Axial_DIN0207_L6.3mm_D2.5mm_P10.16mm_Horizontal -> Resistor_THT:R_Axial_DIN0207_L6.3mm_D2.5mm_P2.54mm_Vertical
Changed lines of the file:
@@
 F 0 "R4" V 2493 2950 50  0000 C CNN
 F 1 "33K" V 2584 2950 50  0000 C CNN
-F 2 "Resistor_THT:R_Axial_DIN0207_L6.3mm_D2.5mm_P2.54mm_Vertical" V 2630 2950 50  0001 C CNN
+F 2 "Resistor_THT:R_Axial_DIN0207_L6.3mm_D2.5mm_P10.16mm_Horizontal" V 2630 2950 50  0001 C CNN
 F 3 "~" H 2700 2950 50  0001 C CNN
 	1    2700 2950
@@
 F 0 "R25" V 9057 1300 50  0000 C CNN
 F 1 "100K" V 8966 1300 50  0000 C CNN
-F 2 "Resistor_THT:R_Axial_DIN0207_L6.3mm_D2.5mm_P10.16mm_Horizontal" V 8780 1300 50  0001 C CNN
+F 2 "Resistor_THT:R_Axial_DIN0207_L6.3mm_D2.5mm_P2.54mm_Vertical" V 8780 1300 50  0001 C CNN
 F 3 "~" H 8850 1300 50  0001 C CNN
 	1    8850 1300
@@
 F 0 "R2" V 2443 6400 50  0000 C CNN
 F 1 "33K" V 2534 6400 50  0000 C CNN
-F 2 "Resistor_THT:R_Axial_DIN0207_L6.3mm_D2.5mm_P2.54mm_Vertical" V 2580 6400 50  0001 C CNN
+F 2 "Resistor_THT:R_Axial_DIN0207_L6.3mm_D2.5mm_P10.16mm_Horizontal" V 2580 6400 50  0001 C CNN
 F 3 "~" H 2650 6400 50  0001 C CNN
 	1    2650 6400
@@
 F 0 "R29" H 10280 2854 50  0000 R CNN
 F 1 "33K" H 10280 2945 50  0000 R CNN
-F 2 "Resistor_THT:R_Axial_DIN0207_L6.3mm_D2.5mm_P10.16mm_Horizontal" V 10280 2900 50  0001 C CNN
+F 2 "Resistor_THT:R_Axial_DIN0207_L6.3mm_D2.5mm_P2.54mm_Vertical" V 10280 2900 50  0001 C CNN
 F 3 "~" H 10350 2900 50  0001 C CNN
 	1    10350 2900
