File: Yusynth_ADSR/yusynth_adsr.kicad_pcb (KiCad board)
At the start: 2 copper layers, 45 x 100 mm, 57 parts, among them Q1 BC547, Q2 BC547, Q3 BC547, Q4 BS170, U1a1 ICM7555xB_SOIC, U1b1 ICM7555xB_DIP, U2 TL074

Commit message: Corrections made after running DRC
Routing:
- net /7555_DIS: track 40.0 -> 41.4 mm
- net /7555_Q: track 23.8 -> 24.9 mm
Other:
- net class Default: trace_width 0.25 -> 0.35

Commit message: Corrections made to ground planes, trace widths, etc. after visual checks of printout
Other:
- net class Power: via_dia 0.8 -> 1; via_drill 0.4 -> 0.5
